File: MiDi.kicad_sch (KiCad schematic)
At the start: 9 parts, among them J1 DIN-5_180degree, J2 Conn_01x06, U2 LTV-356T

Commit message: V1.1
ChangeList

1) Reduce width to 0.8"
2) Reduce TP size (to 0.5mm) move inside edge cut
3) Move J2 closer to edge cut
4) Change Diode footprint to 603.  Old ?SMD_323? was too prone to
	tombstoning
5) Change QR Code.
Parts:
- D1: footprint Diode_SMD:D_SOD-323 -> Diode_SMD:D_0603_1608Metric
- TP1, TP2, TP3: footprint TestPoint:TestPoint_THTPad_D2.0mm_Drill1.0mm -> TestPoint:TestPoint_THTPad_D1.0mm_Drill0.5mm
Changed lines of the file:
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@@
       (effects (font (size 1.27 1.27)) (justify right) hide)
     )
-    (property "Footprint" "TestPoint:TestPoint_THTPad_D2.0mm_Drill1.0mm" (at 73.66 86.36 0)
+    (property "Footprint" "TestPoint:TestPoint_THTPad_D1.0mm_Drill0.5mm" (at 73.66 86.36 0)
       (effects (font (size 1.27 1.27)) hide)
     )
@@
       (effects (font (size 1.27 1.27)) (justify right) hide)
     )
-    (property "Footprint" "TestPoint:TestPoint_THTPad_D2.0mm_Drill1.0mm" (at 83.82 66.04 0)
+    (property "Footprint" "TestPoint:TestPoint_THTPad_D1.0mm_Drill0.5mm" (at 83.82 66.04 0)
       (effects (font (size 1.27 1.27)) hide)
     )
@@
       (effects (font (size 1.27 1.27)) (justify left) hide)
     )
-    (property "Footprint" "Diode_SMD:D_SOD-323" (at 78.74 76.2 0)
+    (property "Footprint" "Diode_SMD:D_0603_1608Metric" (at 78.74 76.2 0)
       (effects (font (size 1.27 1.27)) hide)
     )
@@
       (effects (font (size 1.27 1.27)) (justify right) hide)
     )
-    (property "Footprint" "TestPoint:TestPoint_THTPad_D2.0mm_Drill1.0mm" (at 53.34 86.36 0)
+    (property "Footprint" "TestPoint:TestPoint_THTPad_D1.0mm_Drill0.5mm" (at 53.34 86.36 0)
       (effects (font (size 1.27 1.27)) hide)
     )

Commit message: Modify DIN5 footprint file to work with both prevalent styles of DIN5 connector
Parts:
- J1: footprint StockedComponents:CUI_SDS-50J -> StockedComponents:DIN5_MIDI
Changed lines of the file:
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@@
       (effects (font (size 1.27 1.27)) (justify right))
     )
-    (property "Footprint" "StockedComponents:CUI_SDS-50J" (at 55.88 76.2 0)
+    (property "Footprint" "StockedComponents:DIN5_MIDI" (at 55.88 76.2 0)
       (effects (font (size 1.27 1.27)) hide)
     )
