File: NeoPMOD/NeoPMOD.kicad_sch (KiCad schematic)
At the start: 11 parts, among them J1 Conn_01x06, U1 TPS61022, U2 4492, U3 4492, U4 4492, U5 4492

Commit message: work on schematic
Parts:
- added J2: Conn_01x06, symbol Connector_Generic:Conn_01x06
- added J3: Conn_01x02, symbol Connector_Generic:Conn_01x02
- added U6, U7, U8, U9: 4492, StockedComponents:4492_ADA, symbol StockedComponents:4492
Connections:
- net +3.3V: now also J2.1 (Pin_1)
- net +5V: now also U6.2 (V), U7.2 (V), U8.2 (V), U9.2 (V)
- net GND: now also J2.2 (Pin_2), U6.4 (G), U7.4 (G), U8.4 (G), U9.4 (G)
- net Enable: now reaches J1.6 (Pin_6), U1.5 (EN)
- net Enable: now also J2.6 (Pin_6)
- net at U5.3 (O): now also U6.1 (I)
- net DataIn: now reaches J1.3 (Pin_3), U2.1 (I)
- net Loopback: now reaches J1.4 (Pin_4)
- net Loopback: now also J2.4 (Pin_4), J3.2 (Pin_2)
- new net: J2.3 (Pin_3), J3.1 (Pin_1), U9.3 (O)
- new net: U7.3 (O), U8.1 (I)
- new net: U8.3 (O), U9.1 (I)
- new net: U6.3 (O), U7.1 (I)
- no-connect marks 0 -> 2
Other:
- moved on the sheet: C2, R1, R2, U1
